Commit message: changed urdf

File: src/simulation/urdf/prius.urdf (robot description, URDF)
Before this commit: robot prius, 29 links, 28 joints
Links:
- link chassis: geometry collision box size=1.168381 1.654253 0.272347; collision box size=1.267845 1.116344 0.244286
- link front_left_wheel: geometry collision sphere radius=0.31265; visual mesh filename=package://simulation/meshes/wheel.obj scale=0.01 0.01 0.01
- link front_right_wheel: geometry collision sphere radius=0.31265; visual mesh filename=package://simulation/meshes/wheel.obj scale=0.01 0.01 0.01
- link rear_left_wheel: geometry collision sphere radius=0.31265; visual mesh filename=package://simulation/meshes/wheel.obj scale=0.01 0.01 0.01
- link rear_right_wheel: geometry collision sphere radius=0.31265; visual mesh filename=package://simulation/meshes/wheel.obj scale=0.01 0.01 0.01
- link steering_wheel: geometry visual mesh filename=package://simulation/meshes/steering_wheel.obj scale=0.01 0.01 0.01
